Commit message: Gazebo working & gripper working

File: urdf/xarm7.urdf.xacro (robot description, xacro)
@@ -18,4 +18,5 @@
         <gazebo reference="base_link">
             <material>Gazebo/Red</material> <!-- For Gazebo -->
+            <static>true</static>
         </gazebo>
         <collision>
@@ -282,5 +283,5 @@
         <origin xyz="-0.07 0 0.02" rpy="0 0 0" />
         <axis xyz="1 0 0" />
-        <limit effort="1000.0" velocity="1.0" lower="0.0" upper="0.06" />
+        <limit effort="10.0" velocity="1.0" lower="-0.00001" upper="0.06" />
     </joint>
     <joint name="gripper_right_finger_joint" type="prismatic">
@@ -290,5 +291,5 @@
         <axis xyz="1 0 0" />
         <mimic joint="gripper_left_finger_joint" multiplier="-1.0" />
-        <limit effort="1000.0" velocity="1.0" lower="-0.06" upper="0.0" />
+        <limit effort="10.0" velocity="1.0" lower="-0.06" upper="0.00001" />
     </joint>
 </robot>

File: urdf/xarm7_ros2_control.xacro (robot description, xacro)
@@ -58,12 +58,16 @@
         <joint name="gripper_left_finger_joint">
             <command_interface name="position">
-            <param name="min">-${PI / 2}</param>
+            <param name="min">-0.6</param>
             <param name="max">0.0</param>
+            <param name="initial_value">0.0</param>
             </command_interface>
             <state_interface name="position"/>
         </joint>
         <joint name="gripper_right_finger_joint">
+            <state_interface name="position">
+                <param name="initial_value">0.0</param>
+            </state_interface>
             <param name="mimic">gripper_left_finger_joint</param>
-            <param name="multiplier">-1</param>
+            <param name="multiplier">-1.0</param>
         </joint>
     </ros2_control>
